Commit message: parameters change

File: ROS/kfusion_gazebo/urdf/asus_xtion_pro.urdf.xacro (robot description, xacro)
@@ -6,5 +6,6 @@
   <xacro:property name="M_SCALE" value="0.001"/>
   <xacro:property name="asus_xtion_pro_cam_py" value="0.0205"/>
-  <xacro:property name="asus_xtion_pro_depth_rel_rgb_py" value="0.0270" />
+<!--   <xacro:property name="asus_xtion_pro_depth_rel_rgb_py" value="0.0270" /> -->
+  <xacro:property name="asus_xtion_pro_depth_rel_rgb_py" value="0.0" />
   <xacro:property name="asus_xtion_pro_cam_rel_rgb_py"   value="-0.0220" />
   <!-- Parameterised in part by the values in turtlebot_properties.urdf.xacro -->
